File: circuit-sugoi-tsuyoi-machine.kicad_pcb (KiCad board)
At the start: 2 copper layers, 111 x 86 mm, 56 parts, among them J1 PWR, J10 DIN1, J11 DIN2, J12 DIN3, J13 DIN4, J14 DIN5, J15 AIN1, J16 AIN2, J17 AIN3, J18 AIN4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

Commit message: chore: JLCPCBのPCBA発注用設定・ツールを追加。
Parts:
- D1: value LED -> LED_RED
- D2: value LED -> LED_ORANGE
- D3: value LED -> LED_YELLOW
- D4: value LED -> LED_GREEN
