File: circuit-sugoi-tsuyoi-machine.kicad_pcb (KiCad board)
At the start: 2 copper layers, 111 x 86 mm, 56 parts, among them J1 PWR, J10 DIN1, J11 DIN2, J12 DIN3, J13 DIN4, J14 DIN5, J15 AIN1, J16 AIN2, J17 AIN3, J18 AIN4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

Commit message: feature: MCUをSTM32G473RBT6からSTM32G474RBT6へ変更。
Parts:
- U1: value STM32G473RBTx -> STM32G474RBTx
Changed lines of the file:
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@@
 			(drillshape 0)
 			(scaleselection 1)
-			(outputdirectory "out-v1/")
+			(outputdirectory "out/")
 		)
 	)
@@
 			)
 		)
-		(property "Value" "STM32G473RBTx"
+		(property "Value" "STM32G474RBTx"
 			(at 0 7.4 0)
 			(layer "F.Fab")
@@
 			)
 		)
-		(property "Datasheet" "https://www.st.com/resource/en/datasheet/stm32g473rb.pdf"
+		(property "Datasheet" "https://www.st.com/resource/en/datasheet/stm32g474rb.pdf"
 			(at 0 0 0)
 			(layer "F.Fab")

Commit message: feature: CANトランシーバーをTJA1441ATからATA6561-GAQWへ変更。
Parts:
- U4: value TJA1441AT -> ATA6561-GAQW
Changed lines of the file:
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@@
 			)
 		)
-		(property "Value" "TJA1441AT"
+		(property "Value" "ATA6561-GAQW"
 			(at 0 3.4 0)
 			(layer "F.Fab")
@@
 			)
 		)
-		(property "Datasheet" "http://www.nxp.com/docs/en/data-sheet/TJA1441.pdf"
+		(property "Datasheet" "https://ww1.microchip.com/downloads/aemDocuments/documents/OTH/ProductDocuments/DataSheets/20005991B.pdf"
 			(at 0 0 0)
 			(layer "F.Fab")
@@
 			)
 		)
-		(property "Description" "High-Speed CAN Transceiver, separate VIO, silent mode, SO-8"
+		(property "Description" "High-Speed CAN Transceiver, separate VIO, standby pin, SO-8"
 			(at 0 0 0)
 			(layer "F.Fab")
@@
 			)
 		)
-		(property "LCSC PN" "C3234084"
+		(property "LCSC PN" "C2929602"
 			(at 0 0 0)
 			(unlocked yes)
@@
 			)
 		)
-		(property "LCSC PN" "C529360"
+		(property "LCSC PN" "C529413"
 			(at 0 0 0)
 			(unlocked yes)

Commit message: feature: GNDのベタ塗りを調整。
Routing:
- net LPUART1_RX: track 46.9 -> 58.9 mm
- net LPUART1_TX: track 47.0 -> 59.0 mm
- net AIN3: track 36.4 -> 42.5 mm
- net AIN2: track 39.8 -> 45.8 mm
- net AIN1: track 47.8 -> 53.8 mm
- net AIN4: track 39.4 -> 42.3 mm
- net DIN2: track 28.8 -> 30.5 mm
- net DIN1: track 28.6 -> 30.1 mm
- net GND: vias 78 -> 104
