File: circuit-sugoi-tsuyoi-machine.kicad_sch (KiCad schematic)
At the start: 16 parts, among them SW1 SW_MEC_5E, U1 STM32G473RBTx

Commit message: chore: JLCPCBのPCBA発注用設定・ツールを追加。
Parts:
- C1, C2, C3, C4, C5: LCSC PN (none) -> C14663
- D1: value LED -> LED_RED; LCSC PN (none) -> C84263
- D2: value LED -> LED_ORANGE; LCSC PN (none) -> C84269
- D3: value LED -> LED_YELLOW; LCSC PN (none) -> C84268
- D4: value LED -> LED_GREEN; LCSC PN (none) -> C84264
- R1, R2, R3, R4: LCSC PN (none) -> C2907089
- R5: LCSC PN (none) -> C2907113
- U1: LCSC PN (none) -> C529360
Changed lines of the file:
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@@
+			)
+		)
+		(property "LCSC PN" "C2907089"
+			(at 151.13 90.17 0)
+			(effects
+				(font
+					(size 1.27 1.27)
+				)
 			)
 		)
@@
 			)
 		)
+		(property "LCSC PN" "C2907089"
+			(at 140.97 90.17 0)
+			(effects
+				(font
+					(size 1.27 1.27)
+				)
+			)
+		)
 		(pin "1"
 		)
@@
 			)
 		)
+		(property "LCSC PN" "C14663"
+			(at 123.19 52.07 0)
+			(effects
+				(font
+					(size 1.27 1.27)
+				)
+			)
+		)
 		(pin "1"
 		)
@@
 			)
 		)
+		(property "LCSC PN" "C529360"
+			(at 99.06 107.95 0)
+			(effects
+				(font
+					(size 1.27 1.27)
+				)
+			)
+		)
 		(pin "37"
 		)
@@
 			)
 		)
+		(property "LCSC PN" ""
+			(at 54.61 74.93 0)
+			(effects
+				(font
+					(size 1.27 1.27)
+				)
+			)
+		)
 		(pin "2"
 		)
@@
 			)
 		)
+		(property "LCSC PN" "C14663"
+			(at 134.62 52.07 0)
+			(effects
+				(font
+					(size 1.27 1.27)
+				)
+			)
+		)
 		(pin "2"
 		)
@@
 		(fields_autoplaced yes)
 		(property "Reference" "D2"
-			(at 165.1 98.1074 90)
+			(at 165.1 96.8374 90)
 			(effects
 				(font
@@
 			)
 		)
-		(property "Value" "LED"
-			(at 165.1 100.6474 90)
+		(property "Value" "LED_ORANGE"
+			(at 165.1 99.3774 90)
 			(effects
 				(font
@@
 			)
 		)
+		(property "LCSC PN" "C84269"
+			(at 165.1 101.9174 90)
+			(effects
+				(font
+					(size 1.27 1.27)
+				)
+				(justify right)
+			)
+		)
 		(pin "1"
 		)
@@
 			)
 		)
+		(property "LCSC PN" "C14663"
+			(at 168.91 52.07 0)
+			(effects
+				(font
+					(size 1.27 1.27)
+				)
+			)
+		)
 		(pin "2"
 		)
@@
 			)
 		)
+		(property "LCSC PN" "C2907113"
+			(at 63.5 67.31 0)
+			(effects
+				(font
+					(size 1.27 1.27)
+				)
+			)
+		)
 		(pin "2"
 		)
@@
 		(fields_autoplaced yes)
 		(property "Reference" "D4"
-			(at 144.78 98.1074 90)
+			(at 144.78 96.8374 90)
 			(effects
 				(font
@@
 			)
 		)
-		(property "Value" "LED"
-			(at 144.78 100.6474 90)
+		(property "Value" "LED_GREEN"
+			(at 144.78 99.3774 90)
 			(effects
 				(font
@@
 			)
 		)
+		(property "LCSC PN" "C84264"
+			(at 144.78 101.9174 90)
+			(effects
+				(font
+					(size 1.27 1.27)
+				)
+				(justify right)
+			)
+		)
 		(pin "1"
 		)
@@
 			)
 		)
+		(property "LCSC PN" "C14663"
+			(at 157.48 52.07 0)
+			(effects
+				(font
+					(size 1.27 1.27)
+				)
+			)
+		)
 		(pin "2"
 		)
@@
 			)
 		)
+		(property "LCSC PN" "C2907089"
+			(at 161.29 90.17 0)
+			(effects
+				(font
+					(size 1.27 1.27)
+				)
+			)
+		)
 		(pin "1"
 		)
@@
 		(fields_autoplaced yes)
 		(property "Reference" "D1"
-			(at 175.26 98.1074 90)
+			(at 175.26 96.8374 90)
 			(effects
 				(font
@@
 			)
 		)
-		(property "Value" "LED"
-			(at 175.26 100.6474 90)
+		(property "Value" "LED_RED"
+			(at 175.26 99.3774 90)
 			(effects
 				(font
@@
 			)
 		)
+		(property "LCSC PN" "C84263"
+			(at 175.26 101.9174 90)
+			(effects
+				(font
+					(size 1.27 1.27)
+				)
+				(justify right)
+			)
+		)
 		(pin "1"
 		)
@@
 			)
 		)
+		(property "LCSC PN" "C2907089"
+			(at 171.45 90.17 0)
+			(effects
+				(font
+					(size 1.27 1.27)
+				)
+			)
+		)
 		(pin "1"
 		)
@@
 		(fields_autoplaced yes)
 		(property "Reference" "D3"
-			(at 154.94 98.1074 90)
+			(at 154.94 96.8374 90)
 			(effects
 				(font
@@
 			)
 		)
-		(property "Value" "LED"
-			(at 154.94 100.6474 90)
+		(property "Value" "LED_YELLOW"
+			(at 154.94 99.3774 90)
 			(effects
 				(font
@@
 			)
 		)
+		(property "LCSC PN" "C84268"
+			(at 154.94 101.9174 90)
+			(effects
+				(font
+					(size 1.27 1.27)
+				)
+				(justify right)
+			)
+		)
 		(pin "1"
 		)
@@
 			)
 		)
+		(property "LCSC PN" "C14663"
+			(at 146.05 52.07 0)
+			(effects
+				(font
+					(size 1.27 1.27)
+				)
+			)
+		)

Commit message: feature: MCUをSTM32G473RBT6からSTM32G474RBT6へ変更。
Parts:
- U1: value STM32G473RBTx -> STM32G474RBTx; symbol MCU_ST_STM32G4:STM32G473RBTx -> MCU_ST_STM32G4:STM32G474RBTx
Changed lines of the file:
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@@
 	)
 	(symbol
-		(lib_id "MCU_ST_STM32G4:STM32G473RBTx")
+		(lib_id "MCU_ST_STM32G4:STM32G474RBTx")
 		(at 99.06 107.95 0)
 		(unit 1)
@@
 			)
 		)
-		(property "Value" "STM32G473RBTx"
+		(property "Value" "STM32G474RBTx"
 			(at 103.7433 158.75 0)
 			(effects
@@
 			)
 		)
-		(property "Datasheet" "https://www.st.com/resource/en/datasheet/stm32g473rb.pdf"
+		(property "Datasheet" "https://www.st.com/resource/en/datasheet/stm32g474rb.pdf"
 			(at 99.06 107.95 0)
 			(effects
@@
 		)
 		(property "LCSC PN" "C529360"
-			(at 99.06 107.95 0)
+			(at 103.7433 161.29 0)
 			(effects
 				(font
 					(size 1.27 1.27)
 				)
+				(justify left)
 			)
 		)

Commit message: feature: CANトランシーバーをTJA1441ATからATA6561-GAQWへ変更。
Parts:
- U1: LCSC PN C529360 -> C529413
Changed lines of the file:
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@@
 			)
 		)
-		(property "LCSC PN" "C529360"
+		(property "LCSC PN" "C529413"
 			(at 103.7433 161.29 0)
 			(effects
