File: parts.kicad_sch (KiCad schematic)
At the start: 11 parts, among them U2 AP130-33Y, U3 TJA1441AT, U4 TJA1441AT, Y1 HSE, Y2 LSE

Commit message: chore: JLCPCBのPCBA発注用設定・ツールを追加。
Parts:
- C10, C11, C6, C7, C8, C9: LCSC PN (none) -> C14663
- U2: LCSC PN (none) -> C236803
- U3, U4: LCSC PN (none) -> C3234084
Changed lines of the file:
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@@
+			)
+		)
+		(property "LCSC PN" "C3234084"
+			(at 116.84 50.8 0)
+			(effects
+				(font
+					(size 1.27 1.27)
+				)
 			)
 		)
@@
 			)
 		)
+		(property "LCSC PN" "C14663"
+			(at 107.95 31.75 0)
+			(effects
+				(font
+					(size 1.27 1.27)
+				)
+			)
+		)
 		(pin "2"
 		)
@@
 			)
 		)
+		(property "LCSC PN" ""
+			(at 162.56 59.69 0)
+			(effects
+				(font
+					(size 1.27 1.27)
+				)
+			)
+		)
 		(pin "1"
 		)
@@
 			)
 		)
+		(property "LCSC PN" "C236803"
+			(at 55.88 46.99 0)
+			(effects
+				(font
+					(size 1.27 1.27)
+				)
+			)
+		)
 		(pin "2"
 		)
@@
 			)
 		)
+		(property "LCSC PN" "C14663"
+			(at 107.95 87.63 0)
+			(effects
+				(font
+					(size 1.27 1.27)
+				)
+			)
+		)
 		(pin "2"
 		)
@@
 			)
 		)
+		(property "LCSC PN" "C14663"
+			(at 68.58 53.34 0)
+			(effects
+				(font
+					(size 1.27 1.27)
+				)
+			)
+		)
 		(pin "1"
 		)
@@
 			)
 		)
+		(property "LCSC PN" "C3234084"
+			(at 116.84 106.68 0)
+			(effects
+				(font
+					(size 1.27 1.27)
+				)
+			)
+		)
 		(pin "9"
 		)
@@
 			)
 		)
+		(property "LCSC PN" ""
+			(at 162.56 46.99 0)
+			(effects
+				(font
+					(size 1.27 1.27)
+				)
+			)
+		)
 		(pin "2"
 		)
@@
 			)
 		)
+		(property "LCSC PN" "C14663"
+			(at 95.25 114.3 0)
+			(effects
+				(font
+					(size 1.27 1.27)
+				)
+			)
+		)
 		(pin "1"
 		)
@@
 			)
 		)
+		(property "LCSC PN" "C14663"
+			(at 43.18 53.34 0)
+			(effects
+				(font
+					(size 1.27 1.27)
+				)
+			)
+		)
 		(pin "1"
 		)
@@
 			)
 		)
+		(property "LCSC PN" "C14663"
+			(at 95.25 58.42 0)
+			(effects
+				(font
+					(size 1.27 1.27)
+				)
+			)
+		)

Commit message: feature: CANトランシーバーをTJA1441ATからATA6561-GAQWへ変更。
Parts:
- U3: value TJA1441AT -> ATA6561-GAQW; symbol circuit-sugoi-tsuyoi-machine:TJA1441AT -> circuit-sugoi-tsuyoi-machine:ATA6561-GAQW; LCSC PN C3234084 -> C2929602
Connections:
- net +3.3V: no longer U3.5 (VIO)
- net +5V: no longer U3.3 (VCC)
- net CAN1_N: no longer U3.6 (CANL)
- net CAN1_P: no longer U3.7 (CANH)
- net FDCAN1_RX: no longer U3.4 (RXD)
- net FDCAN1_TX: no longer U3.1 (TXD)
- net GND: no longer U3.2 (GND), U3.8 (S), U3.9 (GND)
Changed lines of the file:
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@@
 	)
 	(symbol
-		(lib_id "circuit-sugoi-tsuyoi-machine:TJA1441AT")
+		(lib_id "circuit-sugoi-tsuyoi-machine:ATA6561-GAQW")
 		(at 116.84 50.8 0)
 		(unit 1)
@@
 			)
 		)
-		(property "Value" "TJA1441AT"
+		(property "Value" "ATA6561-GAQW"
 			(at 118.9833 40.64 0)
 			(effects
@@
 			)
 		)
-		(property "Datasheet" "http://www.nxp.com/docs/en/data-sheet/TJA1441.pdf"
+		(property "Datasheet" "https://ww1.microchip.com/downloads/aemDocuments/documents/OTH/ProductDocuments/DataSheets/20005991B.pdf"
 			(at 116.84 50.8 0)
 			(effects
@@
 			)
 		)
-		(property "Description" "High-Speed CAN Transceiver, separate VIO, silent mode, SO-8"
+		(property "Description" "High-Speed CAN Transceiver, separate VIO, standby pin, SO-8"
 			(at 116.84 50.8 0)
 			(effects
@@
 			)
 		)
-		(property "LCSC PN" "C3234084"
+		(property "LCSC PN" "C2929602"
 			(at 116.84 50.8 0)
 			(effects
